Commit message: Trying to get Ackermann Steering to work

File: install/my_robot_package/share/my_robot_package/dolly.urdf (robot description, URDF)
Before this commit: robot dolly, 8 links, 7 joints
Links:
- removed link caster
- removed link wheel_left_link
- removed link wheel_right_link
- added link back_left_wheel_link, mass 2; collision cylinder length=0.1 radius=0.15; visual cylinder length=0.1 radius=0.15
- added link back_right_wheel_link, mass 2; collision cylinder length=0.1 radius=0.15; visual cylinder length=0.1 radius=.15
- added link front_left_wheel_link, mass 2; collision cylinder length=0.1 radius=0.15; visual cylinder length=0.1 radius=.15
- added link front_right_wheel_link, mass 2; collision cylinder length=0.1 radius=0.15; visual cylinder length=0.1 radius=.15
- link base: geometry collision box size=1.0 0.4 0.1; visual box size=1.0 0.4 0.1
Joints:
- removed joint caster_joint
- removed joint wheel_left_joint
- removed joint wheel_right_joint
- added joint back_left_wheel_joint: type continuous, parent base, child back_left_wheel_link, origin xyz=0.35 -0.25 0.0 rpy=1.57 0.0 0.0, axis 0.0 0.0 1.0
- added joint back_right_wheel_joint: type continuous, parent base, child back_right_wheel_link, origin xyz=0.35 0.25 0.0 rpy=1.57 0.0 0.0, axis 0.0 0.0 1.0
- added joint front_left_wheel_joint: type continuous, parent base, child front_left_wheel_link, origin xyz=-0.35 -0.25 0.0 rpy=1.57 0.0 0.0, axis 0.0 0.0 1.0
- added joint front_right_wheel_joint: type continuous, parent base, child front_right_wheel_link, origin xyz=-0.35 0.25 0.0 rpy=1.57 0.0 0.0, axis 0.0 0.0 1.0
